File: hardware/autokey/autokey.kicad_sch (KiCad schematic)
At the start: 16 parts, among them SW1 KH-6X6X5H-STM, U1 STM32F072CBT6, U2 TLV70033DDCR, U3 10kΩ, X1 X49SM12MSD2SC

Commit message: mod : change hareware solution
Parts:
- removed C1, C2: 1uF, jlc_lib:C0805, symbol jlc_lib:CL21A106KOQNNNE
- removed C3, C4, C5, C6, C9: 100nF, jlc_lib:C0603, symbol jlc_lib:CL10B104KB8NNNC
- removed C7, C8: 22pF, jlc_lib:C0603, symbol jlc_lib:CC0603JRNPO9BN220
- removed F1: SMD1206-020-30, jlc_lib:F1206, symbol jlc_lib:SMD1206-020-30
- removed SW1: KH-6X6X5H-STM, jlc_lib:SW-SMD_4P-L6.0-W6.0-P4.50-LS9.0_H5.0, symbol jlc_lib:KH-6X6X5H-STM
- removed U1: STM32F072CBT6, jlc_lib:LQFP-48_L7.0-W7.0-P0.50-LS9.0-BL, symbol jlc_lib:STM32F072CBT6
- removed U2: TLV70033DDCR, jlc_lib:SOT-23-5_L3.0-W1.7-P0.95-LS2.8-BR, symbol jlc_lib:TLV70033DDCR
- removed U3: 10kΩ, jlc_lib:R0603, symbol jlc_lib:RCA0310KJLF
- removed USB1: XBDM-9101-018, jlc_lib:USB-A-TH_XBDM-9101-018, symbol jlc_lib:XBDM-9101-018
- removed X1: X49SM12MSD2SC, jlc_lib:HC-49S_L11.4-W4.8, symbol jlc_lib:X49SM12MSD2SC
Connections:
- no-connect marks 3 -> 0
Other:
- note removed: "LDO"
- note removed: "USB"
- note removed: "复位"
- note removed: "晶振"
- note removed: "芯片"
- company: autokey -> (none)
- title: autokey_SCH_V1.0_2026-01-20_zhuxx_Confidential -> (none)

Commit message: add: finish the pcb 1.0
Parts:
- added C1, C2: 22pF, jlc_lib:C0603, symbol jlc:CC0603JRNPO9BN220
- added C10, C11, C7: 106, jlc_lib:C0805, symbol jlc:CL21A106KOQNNNE
- added C3, C4, C5, C6, C8, C9: 104, jlc_lib:C0603, symbol jlc:CL10B104KB8NNNC
- added F1: SMD0603-010-15, jlc_lib:F0603, symbol jlc:SMD0603-010-15
- added R1, R3: 0R, jlc_lib:R0603, symbol jlc:0603WAF0000T5E
- added R2: 1M, jlc_lib:R0603, symbol jlc:RC0603JR-071ML
- added R4, R5: 10K, jlc_lib:R0603, symbol jlc:RC0603JR-0710KL
- added R6, R7: 22Ω, jlc_lib:R0603, symbol jlc:0603WAF220JT5E
- added R8: 1.5kΩ, jlc_lib:R0603, symbol jlc:0603WAF1501T5E
- added SW1: KH-6X6X5H-STM, jlc_lib:SW-SMD_4P-L6.0-W6.0-P4.50-LS9.0_H5.0, symbol jlc:KH-6X6X5H-STM
- added U1: STM32F103C8T6, jlc:LQFP-48_L7.0-W7.0-P0.50-LS9.0-BL, symbol jlc:STM32F103C8T6
- added U2: AMS1117-3.3, jlc_lib:SOT-223-3_L6.5-W3.4-P2.30-LS7.0-BR, symbol jlc:AMS1117-3.3
- added USB1: U217-04XN-XXR84, jlc_lib:USB-A-SMD_U217-041N-4BV81, symbol jlc:U217-04XN-XXR84
- added X1: 8M, jlc_lib:HC-49S_L11.4-W4.8-LS12.7, symbol jlc:H6OEL89CSC-STUYLC-8M
Connections:
- new net: R1.2, U1.1 (VBAT)
- new net: R4.2, U1.20 (PB2)
- new net: R5.2, U1.44 (BOOT0)
- new net: C1.2, R2.2, U1.5 (PD0-OSC_IN), X1.2 (OSC2)
- new net: C2.2, R2.1, U1.6 (PD1-OSC_OUT), X1.1 (OSC1)
- new net: R3.2, U1.9 (VDDA)
- new net: R7.1, R8.1, USB1.3 (D+)
- new net: F1.1, USB1.1 (VCC)
- new net: R6.1, USB1.2 (D-)
- new net +3.3V: C11.2, C3.2, C4.2, C5.2, C6.2, C7.2, C8.2, R1.1, R3.1, R8.2, U1.24 (VDD_1), U1.36 (VDD_2), U1.48 (VDD_3), U2.4 (VOUT)
- new net +5V: C10.1, C9.2, F1.2, U2.3 (VIN)
- new net GND: C1.1, C10.2, C11.1, C2.1, C3.1, C4.1, C5.1, C6.1, C7.1, C8.1, C9.1, R4.1, R5.1, SW1.2, U1.23 (VSS_1), U1.35 (VSS_2), U1.47 (VSS_3), U1.8 (VSSA), U2.1 (GND), USB1.4 (GND), USB1.5, USB1.6
- new net PA1: SW1.3, U1.11 (PA1)
- new net USB_DM: R6.2, U1.32 (PA11)
- new net USB_DP: R7.2, U1.33 (PA12)
